File: stackmat-pcb/stackmat.kicad_sch (KiCad schematic)
At the start: 14 parts, among them U2 18650, U3 AMS1117-3.3

Commit message: feat: hardware based serial amplifier, better submit button
Connections:
- net +3.3V: now also NPN1.3 (E); no longer NPN1.1 (C)
- net at JF1.2 (Pin_2): now also NPN1.1 (C); no longer NPN1.3 (E)
Changed lines of the file:
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@@
+    (stroke (width 0) (type default))
+  )
+  (wire (pts (xy 194.31 58.42) (xy 203.2 58.42))
+    (stroke (width 0) (type default))
+  )
+  (wire (pts (xy 180.34 36.83) (xy 194.31 36.83))
     (stroke (width 0) (type default))
   )
@@
     (stroke (width 0) (type default))
   )
+  (wire (pts (xy 194.31 36.83) (xy 194.31 58.42))
+    (stroke (width 0) (type default))
+  )
   (wire (pts (xy 162.56 125.73) (xy 162.56 129.54))
     (stroke (width 0) (type default))
   )
-  (wire (pts (xy 180.34 58.42) (xy 203.2 58.42))
-    (stroke (width 0) (type default))
-  )
   (wire (pts (xy 172.72 41.91) (xy 172.72 55.88))
     (stroke (width 0) (type default))
@@
   )
   (wire (pts (xy 140.97 54.61) (xy 140.97 68.58))
-    (stroke (width 0) (type default))
-  )
-  (wire (pts (xy 180.34 46.99) (xy 180.34 58.42))
     (stroke (width 0) (type default))
   )
@@
     )
   )
-  (symbol (lib_id "power:+3.3V") (at 180.34 36.83 0) (unit 1)
-    (in_bom yes) (on_board yes) (dnp no) (fields_autoplaced)
-    (property "Reference" "#PWR01" (at 180.34 40.64 0)
-      (effects (font (size 1.27 1.27)) hide)
-    )
-    (property "Value" "+3.3V" (at 180.34 31.75 0)
-      (effects (font (size 1.27 1.27)))
-    )
-    (property "Footprint" "" (at 180.34 36.83 0)
-      (effects (font (size 1.27 1.27)) hide)
-    )
-    (property "Datasheet" "" (at 180.34 36.83 0)
-      (effects (font (size 1.27 1.27)) hide)
-    )
+  (symbol (lib_id "power:+3.3V") (at 180.34 46.99 180) (unit 1)
+    (in_bom yes) (on_board yes) (dnp no) (fields_autoplaced)
+    (property "Reference" "#PWR01" (at 180.34 43.18 0)
+      (effects (font (size 1.27 1.27)) hide)
+    )
+    (property "Value" "+3.3V" (at 182.88 48.26 0)
+      (effects (font (size 1.27 1.27)) (justify right))
+    )
+    (property "Footprint" "" (at 180.34 46.99 0)
+      (effects (font (size 1.27 1.27)) hide)
+    )
+    (property "Datasheet" "" (at 180.34 46.99 0)
+      (effects (font (size 1.27 1.27)) hide)
+    )

Commit message: feat: delegate button
Parts:
- removed BTN1: Conn_01x03, Connector_PinHeader_2.54mm:PinHeader_1x03_P2.54mm_Vertical, symbol Connector_Generic:Conn_01x03
- added BTN1: Conn_01x05, Connector_PinHeader_2.54mm:PinHeader_1x05_P2.54mm_Vertical, symbol Connector_Generic:Conn_01x05
- R2: value R100000 -> R10000
Connections:
- net +3.3V: now also BTN1.2 (Pin_2)
- net GND: now also BTN1.1 (Pin_1)
- net at ESP12f1.16 (GPIO15), R1.1: now also BTN1.5 (Pin_5); no longer RFID1.3 (Pin_3)
- net at ESP12f1.17 (GPIO2): now also BTN1.3 (Pin_3)
- net at ESP12f1.18 (GPIO0): now also BTN1.4 (Pin_4)
- net at ESP12f1.4 (GPIO16): now also RFID1.3 (Pin_3)
Changed lines of the file:
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@@
   (junction (at 140.97 68.58) (diameter 0) (color 0 0 0 0)
   )
+  (junction (at 157.48 99.06) (diameter 0) (color 0 0 0 0)
+  )
   (junction (at 172.72 63.5) (diameter 0) (color 0 0 0 0)
   )
   (junction (at 165.1 83.82) (diameter 0) (color 0 0 0 0)
   )
-  (junction (at 162.56 99.06) (diameter 0) (color 0 0 0 0)
-  )
   (junction (at 63.5 91.44) (diameter 0) (color 0 0 0 0)
   )
@@
     (stroke (width 0) (type default))
   )
-  (wire (pts (xy 163.83 129.54) (xy 165.1 129.54))
+  (wire (pts (xy 163.83 123.19) (xy 162.56 123.19))
     (stroke (width 0) (type default))
   )
@@
     (stroke (width 0) (type default))
   )
-  (wire (pts (xy 162.56 125.73) (xy 162.56 129.54))
+  (wire (pts (xy 160.02 125.73) (xy 160.02 129.54))
+    (stroke (width 0) (type default))
+  )
+  (wire (pts (xy 157.48 99.06) (xy 162.56 99.06))
     (stroke (width 0) (type default))
   )
@@
     (stroke (width 0) (type default))
   )
+  (wire (pts (xy 156.21 101.6) (xy 156.21 109.22))
+    (stroke (width 0) (type default))
+  )
+  (wire (pts (xy 185.42 99.06) (xy 181.61 99.06))
+    (stroke (width 0) (type default))
+  )
+  (wire (pts (xy 181.61 109.22) (xy 156.21 109.22))
+    (stroke (width 0) (type default))
+  )
   (wire (pts (xy 77.47 99.06) (xy 80.01 99.06))
     (stroke (width 0) (type default))
   )
+  (wire (pts (xy 157.48 99.06) (xy 157.48 129.54))
+    (stroke (width 0) (type default))
+  )
+  (wire (pts (xy 163.83 81.28) (xy 163.83 123.19))
+    (stroke (width 0) (type default))
+  )
   (wire (pts (xy 80.01 91.44) (xy 73.66 91.44))
     (stroke (width 0) (type default))
   )
+  (wire (pts (xy 162.56 123.19) (xy 162.56 129.54))
+    (stroke (width 0) (type default))
+  )
   (wire (pts (xy 173.99 86.36) (xy 173.99 87.63))
     (stroke (width 0) (type default))
@@
     (stroke (width 0) (type default))
   )
+  (wire (pts (xy 181.61 99.06) (xy 181.61 109.22))
+    (stroke (width 0) (type default))
+  )
   (wire (pts (xy 172.72 63.5) (xy 203.2 63.5))
     (stroke (width 0) (type default))
@@
     (stroke (width 0) (type default))
   )
-  (wire (pts (xy 162.56 99.06) (xy 185.42 99.06))
-    (stroke (width 0) (type default))
-  )
   (wire (pts (xy 73.66 74.93) (xy 76.2 74.93))
     (stroke (width 0) (type default))
@@
     (stroke (width 0) (type default))
   )
-  (wire (pts (xy 156.21 99.06) (xy 162.56 99.06))
+  (wire (pts (xy 156.21 99.06) (xy 157.48 99.06))
     (stroke (width 0) (type default))
   )
@@
     (stroke (width 0) (type default))
   )
-  (wire (pts (xy 162.56 125.73) (xy 203.2 125.73))
+  (wire (pts (xy 160.02 125.73) (xy 203.2 125.73))
     (stroke (width 0) (type default))
   )
@@
   )
   (wire (pts (xy 156.21 86.36) (xy 173.99 86.36))
-    (stroke (width 0) (type default))
-  )
-  (wire (pts (xy 163.83 81.28) (xy 163.83 129.54))
     (stroke (width 0) (type default))
   )
@@
         (path "/ccd0dcac-df1d-4089-8f7e-e62a3e2f6f2a"
           (reference "#PWR0103") (unit 1)
+        )
+      )
+    )
+  )
+  (symbol (lib_id "Connector_Generic:Conn_01x05") (at 162.56 134.62 270) (unit 1)
+    (in_bom yes) (on_board yes) (dnp no) (fields_autoplaced)
+    (property "Reference" "BTN1" (at 162.56 138.43 90)
+      (effects (font (size 1.27 1.27)))
+    )
+    (property "Value" "Conn_01x05" (at 162.56 140.97 90)
+      (effects (font (size 1.27 1.27)) hide)
+    )
+    (property "Footprint" "Connector_PinHeader_2.54mm:PinHeader_1x05_P2.54mm_Vertical" (at 162.56 134.62 0)
+      (effects (font (size 1.27 1.27)) hide)
+    )
+    (property "Datasheet" "~" (at 162.56 134.62 0)
+      (effects (font (size 1.27 1.27)) hide)
+    )
+    (pin "1")
+    (pin "4")
+    (pin "5")
+    (pin "2")
+    (pin "3")
+    (instances
+      (project "stackmat"
+        (path "/ccd0dcac-df1d-4089-8f7e-e62a3e2f6f2a"
+          (reference "BTN1") (unit 1)
+        )
+      )
+    )
+  )
+  (symbol (lib_id "power:+3.3V") (at 165.1 129.54 0) (unit 1)
+    (in_bom yes) (on_board yes) (dnp no) (fields_autoplaced)
+    (property "Reference" "#PWR02" (at 165.1 133.35 0)
+      (effects (font (size 1.27 1.27)) hide)
+    )
+    (property "Value" "+3.3V" (at 165.1 124.46 0)
+      (effects (font (size 1.27 1.27)))
+    )
+    (property "Footprint" "" (at 165.1 129.54 0)
+      (effects (font (size 1.27 1.27)) hide)
+    )
+    (property "Datasheet" "" (at 165.1 129.54 0)
+      (effects (font (size 1.27 1.27)) hide)
+    )
+    (pin "1")
+    (instances
+      (project "stackmat"
+        (path "/ccd0dcac-df1d-4089-8f7e-e62a3e2f6f2a"
+          (reference "#PWR02") (unit 1)
         )
       )
@@
     )
   )
-  (symbol (lib_id "Connector_Generic:Conn_01x03") (at 165.1 134.62 270) (unit 1)
-    (in_bom yes) (on_board yes) (dnp no)
-    (property "Reference" "BTN1" (at 162.56 137.16 90)
-      (effects (font (size 1.27 1.27)) (justify left))
-    )
-    (property "Value" "Conn_01x03" (at 170.18 135.89 90)
-      (effects (font (size 1.27 1.27)) (justify left))
-    )
-    (property "Footprint" "Connector_PinHeader_2.54mm:PinHeader_1x03_P2.54mm_Vertical" (at 165.1 134.62 0)
-      (effects (font (size 1.27 1.27)) hide)
-    )
-    (property "Datasheet" "~" (at 165.1 134.62 0)
-      (effects (font (size 1.27 1.27)) hide)
-    )
-    (pin "3")
-    (pin "2")
-    (pin "1")
-    (instances
-      (project "stackmat"
-        (path "/ccd0dcac-df1d-4089-8f7e-e62a3e2f6f2a"
-          (reference "BTN1") (unit 1)
-        )
-      )
-    )
-  )
   (symbol (lib_id "Connector_Generic:Conn_01x04") (at 190.5 83.82 0) (unit 1)
     (in_bom yes) (on_board yes) (dnp no)
@@
   (symbol (lib_id "Device:R") (at 172.72 59.69 0) (unit 1)
     (in_bom yes) (on_board yes) (dnp no) (fields_autoplaced)
-    (property "Reference" "R2" (at 175.26 58.4199 0)
-      (effects (font (size 1.27 1.27)) (justify left))
-    )
-    (property "Value" "R100000" (at 175.26 60.9599 0)
-      (effects (font (size 1.27 1.27)) (justify left))
-    )
+    (property "Reference" "R2" (at 175.26 58.42 0)
+      (effects (font (size 1.27 1.27)) (justify left))
+    )
+    (property "Value" "R10000" (at 175.26 60.96 0)
+      (effects (font (size 1.27 1.27)) (justify left))
+    )
